File: schematic/REGO600/REGO600.kicad_sch (KiCad schematic)
At the start: 39 parts, among them J1 RJ45, J10 HP, J11 GT11, J12 GT10, J13 GT8, J14 GT6, J15 GT3, J16 GT9, J17 GT3, J18 EXT, J19 SUMMA LARM, J2 Conn_02x13_Odd_Even, J20 GT5, J21 GT4, J22 ALARM_LED, J23 GT3X, J24 GT1, J25 GT2, J3 Conn_02x13_Odd_Even, J4 Conn_02x08_Odd_Even, J5 Conn_02x05_Odd_Even, J6 Conn_02x05_Odd_Even, J7 Conn_02x08_Odd_Even, J8 DE9_Pins_MountingHoles, J9 LP, U2 SP720, U3 CY62256-70PC, U4 27512, U5 74HC373, U6 SST39SF040, Y1 Crystal

Commit message: update schematic
Parts:
- added C3: C_Polarized, symbol Device:C_Polarized
- added C4, C5, C6: C, symbol Device:C
- added J26: ToRelayBoard, Connector_PinHeader_2.54mm:PinHeader_2x13_P2.54mm_Horizontal, symbol Connector_Generic:Conn_02x13_Odd_Even
- added R10, R11, R9: 100k, symbol Device:R
- added R12, R13, R14: 1M, symbol Device:R
- added R15, R16, R17, R18, R19, R20, R21, R22, R23: 470, symbol Device:R
- added R6, R7, R8: 470k, symbol Device:R
- added U10, U9: CD4051B, symbol Analog_Switch:CD4051B
- added U11, U12: 4049, symbol 4xxx:4049
- added U13: 40106, symbol 4xxx:40106
- added U14: 4021, symbol 4xxx:4021
- added U15: DS1302Z+, Package_SO:SOIC-8_3.9x4.9mm_P1.27mm, symbol Timer_RTC:DS1302Z+
- added U16: SP720, Package_SO:SOIC-16_3.9x9.9mm_P1.27mm, symbol IC_Automotive:SP720
- added U7, U8: HEF4094B, symbol 4xxx:HEF4094B
- added Y2: Crystal, symbol Device:Crystal
Connections:
- net +5V: now also J26.25 (Pin_25), J26.26 (Pin_26), R6.1, R7.1, R8.1, U14.16 (VDD)
- net GND: now also C4.2, C5.2, C6.2, J26.1 (Pin_1), J26.2 (Pin_2), R10.2, R11.2, R9.2, U14.8 (VSS)
- net 4021.LATCH: now reaches U1.12 (P4.5/CMSR5)
- net 4021.LATCH: now also U14.9 (PL)
- net 4021.CLK: now reaches U1.14 (P4.7/CMT1)
- net 4021.CLK: now also U14.10 (CP)
- net 4021.DAT: now reaches U1.21 (P1.5/RT2)
- net 4021.DAT: now also U14.3 (Q7)
- new net: R14.2, U13.1
- new net: U13.2, U14.15 (D6)
- new net: C4.1, J26.4 (Pin_4), R6.2, U14.6 (D1)
- new net: J26.22 (Pin_22), R20.2
- new net: J26.11 (Pin_11), R10.1, R13.1
- new net: C6.1, J26.6 (Pin_6), R8.2, U14.4 (D3)
- new net: J26.17 (Pin_17), R18.1
- new net: C5.1, J26.5 (Pin_5), R7.2, U14.5 (D2)
- new net: R13.2, U13.3
- new net: J26.18 (Pin_18), R22.2
- new net: J26.13 (Pin_13), R12.1, R9.1
- new net: J26.20 (Pin_20), R21.2
- new net: J26.16 (Pin_16), R23.2
- new net: J26.23 (Pin_23), R15.1
- new net: J26.9 (Pin_9), R11.1, R14.1
- new net: U13.4, U14.14 (D5)
- new net: R12.2, U13.5
- new net: U13.6, U14.13 (D4)
- new net: J26.21 (Pin_21), R16.1
- new net: J26.19 (Pin_19), R17.1
- new net: J26.24 (Pin_24), R19.2
