File: schematic/REGO600/REGO600.kicad_sch (KiCad schematic)
At the start: 73 parts, among them J1 RJ45, J10 HP, J11 GT11, J12 GT10, J13 GT8, J14 GT6, J15 GT3, J16 GT9, J17 GT3, J18 EXT, J19 SUMMA LARM, J2 Conn_02x13_Odd_Even, J20 GT5, J21 GT4, J22 ALARM_LED, J23 GT3X, J24 GT1, J25 GT2, J26 ToRelayBoard, J3 Conn_02x13_Odd_Even, J4 Conn_02x08_Odd_Even, J5 Conn_02x05_Odd_Even, J6 Conn_02x05_Odd_Even, J7 Conn_02x08_Odd_Even, J8 DE9_Pins_MountingHoles, J9 LP, U10 CD4051B, U11 4049, U12 4049, U13 40106, U14 4021, U15 DS1302Z+, U16 SP720, U2 SP720, U3 CY62256-70PC, U4 27512, U5 74HC373, U6 SST39SF040, U7 HEF4094B, U8 HEF4094B, U9 CD4051B, Y1 Crystal, Y2 Crystal

Commit message: update schema
Parts:
- added R24, R25, R26, R27, R28, R29, R30, R31, R32: 47k, symbol Device:R
Connections:
- net +5V: now also R24.1, R25.1, R26.1, R27.1, R28.1, R29.1, R30.1, R31.1, R32.1
- net at U12.14: now also R32.2
- net at U12.15: now also R18.2
- net at U12.2: now also R20.1
- net at U12.3: now also R25.2
- net at U11.2: now also R22.1
- net at U11.3: now also R27.2
- net at U11.4: now also R23.1
- net at U11.5: now also R28.2
- net at U11.14: now also R30.2
- net at U11.15: now also R16.2
- net at U12.10: now also R15.2
- net at U12.9: now also R29.2
- net at R21.1: now also U11.12
- net at U12.11: now also R24.2
- net at U12.12: now also R19.1
- net at U11.11: now also R26.2
- net at R17.2: now also U11.10
- net at U11.9: now also R31.2
Other:
- moved on the sheet: C4, C5, C6, J26, R10, R11, R12, R13, R14, R15, R16, R17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

Commit message: schema now done for CPU PCB
Parts:
- removed C4, C5, C6: C, symbol Device:C
- removed J2: Conn_02x13_Odd_Even, Connector_IDC:IDC-Header_2x13_P2.54mm_Latch_Horizontal, symbol Connector_Generic:Conn_02x13_Odd_Even
- removed R6, R7, R8: 470k, symbol Device:R
- added C10, C11, C12, C13, C14, C15, C16, C17, C18, C19, C20, C21, C22, C23, C24, C25, C26, C27, C28, C29, C30, C31, C32, C33, C34, C35, C36, C37, C38, C39, C40, C41, C42, C8, C9: C, symbol Device:C
- added J27: SIGNAL I/O, Connector_IDC:IDC-Header_2x13_P2.54mm_Latch_Horizontal, symbol Connector_Generic:Conn_02x13_Odd_Even
- added K1: G5V-2, Relay_THT:Relay_DPDT_Omron_G5V-2, symbol Relay:G5V-2
- added Q1: BC847, Package_TO_SOT_SMD:SOT-23, symbol Transistor_BJT:BC847
- added R33, R34: 2k7, symbol Device:R
- added R35, R36, R37, R38, R39, R40, R41, R42, R43, R44, R45, R46, R47, R48, R49, R50, R67: 10k, symbol Device:R
- added R51, R52, R53, R54, R55, R56, R57, R58, R59, R60, R61, R62, R63, R64, R65, R66: 4k7, symbol Device:R
- added R68, R69, R70: 470k, symbol Device:R
- added U17: (no value), Package_SO:SOIC-8_5.3x5.3mm_P1.27mm, symbol TC1232:TC1232
- C3: value C_Polarized -> 0F1
- J26: value ToRelayBoard -> ToPowerBoard
- Y1: value Crystal -> 11050000
- Y2: value Crystal -> 32k
Connections:
- net +5V: now also C3.1, U1.59 (AVref+), U1.61 (AVdd), U10.16 (VDD), U11.1 (VCC), U12.1 (VCC), U13.14 (VDD), U15.1 (VCC2), U15.8 (VCC1), U16.16 (V+), U7.16 (V_{DD}), U8.16 (V_{DD}), U9.16 (VDD), J27.13 (Pin_13), K1.1, R51.1, R52.1, R53.1, R54.1, R55.1, R56.1, R57.1, R58.1, R59.1, R60.1, R61.1, R62.1, R63.1, R64.1, R65.1, R66.1, R68.1, R69.1, R70.1, U17.2 (TD), U17.3 (TOL), U17.8 (Vcc)
- net GND: now also C3.2, U1.3 (STADC), U1.58 (AVref-), U1.6 (EW#), U1.60 (AVss), U10.7 (VEE), U10.8 (VSS), U11.8 (VSS), U12.8 (VSS), U13.7 (VSS), U15.4 (GND), U16.8 (GND), U7.8 (V_{SS}), U8.8 (V_{SS}), U9.7 (VEE), U9.8 (VSS), C10.2, C11.2, C12.2, C13.2, C14.2, C15.2, C16.2, C17.2, C18.2, C19.2, C20.2, C21.2, C22.2, C23.2, C24.2, C25.2, C26.2, C27.2, C28.2, C29.2, C30.2, C31.2, C32.2, C33.2, C34.2, C35.2, C36.2, C37.2, C38.2, C39.2, C40.2, C41.2, C42.2, C8.2, C9.2, J27.16 (Pin_16), J27.26 (Pin_26), Q1.2 (E), U17.4 (GND)
- net TC1232_STB/DS1302_CS: now also U15.5 (CE), U17.7 (ST#)
- net LARM_LED: now reaches U12.4
- net LARM_LED: now also U2.11 (I10), J27.22 (Pin_22)
- net at U12.5: now also U8.12 (QP6)
- net ALE#: now reaches U1.48 (ALE), U5.11 (LE)
- net DISPLAY_~{INT#}: now reaches J1.3, R1.2, U1.26 (P3.2/INT#)
- net 4094.LATCH: now reaches U8.1 (STR)
- net 4094.LATCH: now also U1.11 (P4.4/CMSR4), U7.1 (STR)
- net at U8.11 (QP7): now also U12.7
- net 4094.B.EL6: now reaches U8.13 (QP5)
- net 4094.B.EL6: now also R28.2, U11.5
- net SUMMA_LARM_RELAY: now reaches U8.14 (QP4)
- net SUMMA_LARM_RELAY: now also R67.1
- net at U8.15 (OE): now also U13.10, U7.15 (OE)
- net at U8.2 (D): now also U7.9 (QS1)
- net 4094.CLK: now reaches U8.3 (CP)
- net 4094.CLK: now also U1.19 (P1.3/CT3I), U15.7 (SCLK), U7.3 (CP)
- net 4051_SEL_A: now reaches U8.4 (QP0)
- net 4051_SEL_A: now also U10.11 (A), U9.11 (A)
- net 4051_SEL_B: now reaches U8.5 (QP1)
- net 4051_SEL_B: now also U10.10 (B), U9.10 (B)
- net 4051_SEL_C: now reaches U8.6 (QP2)
- net 4051_SEL_C: now also U10.9 (C), U9.9 (C)
- net 4051_SEL_(C)_INH: now reaches U8.7 (QP3)
- net 4051_SEL_(C)_INH: now also U13.9, U9.6 (INH)
- net 4094.A.P3: now reaches R29.2, U12.9
- net 4094.A.P3: now also U7.11 (QP7)
- net 4094.A.EL3: now reaches R32.2, U12.14
- net 4094.A.EL3: now also U7.6 (QP2)
- net 4094.A.s2: now reaches R26.2, U11.11
- net 4094.A.s2: now also U7.5 (QP1)
- net 4094.A.P2: now reaches R30.2, U11.14
- net 4094.A.P2: now also U7.13 (QP5)
- net 4094.A.VXV: now reaches R25.2, U12.3
- net 4094.A.VXV: now also U7.14 (QP4)
- net at J26.4 (Pin_4), U14.6 (D1): now also C40.1, R68.2
- net DISPLAY_I2C_SDA: now reaches J1.4, R3.2, R5.1
- net DISPLAY_I2C_SDA: now also U2.2 (I2)
- net at Y2.1: now also U15.2 (X1)
- net at Y2.2: now also U15.3 (X2)
- net at J26.6 (Pin_6), U14.4 (D3): now also C42.1, R70.2
- net 4094.A.P1: now reaches R27.2, U11.3
- net 4094.A.P1: now also U7.7 (QP3)
- net at U1.1 (P5.0/ADC0): now also U10.3 (X), U9.3 (X)
- net at U1.15 (RST): now also U17.5 (RST)
- net DS1302_IO: now reaches U1.17 (P1.1/CT1I)
- net DS1302_IO: now also U15.6 (I/O)
- net 4094.DAT: now reaches U1.20 (P1.4/T2)
- net 4094.DAT: now also U7.2 (D)
- net at U1.24 (P3.0/RxD): now also U13.13, R33.2
- net at U1.25 (P3.1/TxD): now also U11.7
- net WR#: now reaches U1.30 (P3.6/WR#), U3.27 (~{WE}), U6.31 (PGM)
- net RD#: now reaches U1.31 (P3.7/RD#), U3.22 (~{OE}), U6.24 (OE)
- net 4094.OE: now reaches U1.4 (PWM0#)
- net 4094.OE: now also U13.11
- net PSEN#: now reaches U1.47 (PSEN#), U4.22 (~{OE})
- net DISPLAY_I2C_SCL: now reaches J1.5, R2.2, R4.1
- net DISPLAY_I2C_SCL: now also U2.6 (I6)
- net at J26.5 (Pin_5), U14.5 (D2): now also C41.1, R69.2
- net EXT_CTRL: now reaches U16.1 (I1)
- net EXT_CTRL: now also C31.1, J27.17 (Pin_17), R42.2, R58.2
- net HP: now reaches U16.10 (I9)
- net HP: now also C39.1, J27.4 (Pin_4), R43.2, R66.2
- net SERVICE_ADC: now reaches U16.11 (I10)
- net SERVICE_ADC: now also C38.1, J27.9 (Pin_9), R44.2, R65.2
- net GT10: now reaches U16.12 (I11)
- net GT10: now also C37.1, J27.8 (Pin_8), R45.2, R64.2
- net GT8: now reaches U16.13 (I12)
- net GT8: now also C36.1, J27.10 (Pin_10), R46.2, R63.2
- net GT6: now reaches U16.14 (I13)
- net GT6: now also C35.1, J27.12 (Pin_12), R47.2, R62.2
- net GT3: now reaches U16.15 (I14)
- net GT3: now also C34.1, J27.14 (Pin_14), R48.2, R61.2
- net GT5: now reaches U16.2 (I2)
- net GT5: now also C30.1, J27.19 (Pin_19), R41.2, R57.2
- net GT4: now reaches U16.3 (I3)
- net GT4: now also C29.1, J27.21 (Pin_21), R40.2, R56.2
- net GT11: now reaches U16.4 (I4)
- net GT11: now also C28.1, J27.6 (Pin_6), R39.2, R55.2
- net GT3X: now reaches U16.5 (I5)
- net GT3X: now also C27.1, J27.23 (Pin_23), R38.2, R54.2
- net GT1: now reaches U16.6 (I6)
- net GT1: now also C26.1, J27.24 (Pin_24), R37.2, R53.2
- net GT2: now reaches U16.7 (I7)
- net GT2: now also C25.1, J27.25 (Pin_25), R36.2, R52.2
- net LP: now reaches U16.9 (I8)
- net LP: now also C24.1, J27.2 (Pin_2), R35.2, R51.2
- net at U10.1 (X4): now also C19.1, R47.1
- net at U10.12 (X3): now also C20.1, R46.1
- net at U10.13 (X0): now also C23.1, R43.1
- net at U10.14 (X1): now also C22.1, R44.1
- net at U10.15 (X2): now also C21.1, R45.1
- net at U10.2 (X6): now also C17.1, R49.1
- net at U10.4 (X7): now also C16.1, R50.1
- net at U10.5 (X5): now also C18.1, R48.1
- net at U10.6 (INH): now also U13.8
- net RxD: now reaches U2.1 (I1)
- net RxD: now also J27.11 (Pin_11), R33.1
- net ALLWAYS_LOW: now reaches U2.10 (I9)
- net ALLWAYS_LOW: now also U12.6, J27.1 (Pin_1)
- net VVP: now reaches U2.15 (I14)
- net VVP: now also C33.1, J27.15 (Pin_15), R49.2, R60.2
- net GT9: now reaches U2.3 (I3)
- net GT9: now also C32.1, J27.7 (Pin_7), R50.2, R59.2
- net TxD: now reaches U2.4 (I4)
- net TxD: now also J27.5 (Pin_5), R34.1
- net DISPLAY_INT: now reaches U2.5 (I5)
- net 4094.A.COMP: now reaches R24.2, U12.11
- net 4094.A.COMP: now also U7.12 (QP6)
- net 4094.A.s1: now reaches U7.4 (QP0)
- net 4094.A.s1: now also R31.2, U11.9
- net at U11.6: now also R34.2
- net at U9.1 (X4): now also C11.1, R38.1
- net at U9.12 (X3): now also C12.1, R39.1
- net at U9.13 (X0): now also C15.1, R42.1
- net at U9.14 (X1): now also C14.1, R41.1
- net at U9.15 (X2): now also C13.1, R40.1
- net at U9.2 (X6): now also C9.1, R36.1
- net at U9.4 (X7): now also C8.1, R35.1
- net at U9.5 (X5): now also C10.1, R37.1
- new net: Q1.1 (B), R67.2
- new net: K1.16, Q1.3 (C)
- new net SUM_LARM_X1: J27.18 (Pin_18), K1.13
- new net SUM_LARM_X2: J27.20 (Pin_20), K1.9
Other:
- note added: "Connected to unpopulated PCB SMD pad"
- note added: "External Sensors/Ext Ctrl Inp/Larm Output - PCB"
- note added: "FLEX_CABLE"
- note added: "Internal Sensors/Service Port - PCB"
- note added: "NC"
- moved on the sheet: C3, J1, J10, J11, J12, J13, J14, J15, J16, J17, J18, J19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
