File: schematic/REGO600/REGO600.kicad_sch (KiCad schematic)
At the start: 152 parts, among them J1 RJ45, J10 HP, J11 GT11, J12 GT10, J13 GT8, J14 GT6, J15 GT3, J16 GT9, J17 GT3, J18 EXT, J19 SUMMA LARM, J20 GT5, J21 GT4, J22 ALARM_LED, J23 GT3X, J24 GT1, J25 GT2, J26 ToPowerBoard, J27 SIGNAL I/O, J3 Conn_02x13_Odd_Even, J4 Conn_02x08_Odd_Even, J5 Conn_02x05_Odd_Even, J6 Conn_02x05_Odd_Even, J7 Conn_02x08_Odd_Even, J8 DE9_Pins_MountingHoles, J9 LP, K1 G5V-2, Q1 BC847, U10 CD4051B, U11 4049, U12 4049, U13 40106, U14 4021, U15 DS1302Z+, U16 SP720, U2 SP720, U3 CY62256-70PC, U4 27512, U5 74HC373, U6 SST39SF040, U7 HEF4094B, U8 HEF4094B, U9 CD4051B, Y1 11050000, Y2 32k

Commit message: simulator now executes whole firmware and LCD and RTC functionality is working, however there is still some hardware to be simulated such as, front panel buttons/leds, phase detection, actuator outputs, sensor inputs and service uart
Parts:
- C3: value 0F1 -> 0F1 SUPERCAP
- U17: value (none) -> TC1232
Connections:
- net +5V: no longer C3.1, U15.8 (VCC1)
- new net: C3.1, U15.8 (VCC1)
Other:
- moved on the sheet: C3
Changed lines of the file:
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@@
 	)
 	(junction
-		(at 62.992 89.408)
-		(diameter 0)
-		(color 0 0 0 0)
-	)
-	(junction
 		(at 491.49 78.74)
 		(diameter 0)
@@
 	)
 	(junction
-		(at 62.992 88.138)
-		(diameter 0)
-		(color 0 0 0 0)
-	)
-	(junction
 		(at 568.96 232.41)
 		(diameter 0)
@@
 	(wire
 		(pts
-			(xy 429.26 97.79) (xy 438.15 97.79)
+			(xy 81.026 102.616) (xy 95.504 102.616)
 		)
 		(stroke
@@
 	(wire
 		(pts
-			(xy 195.58 212.09) (xy 195.58 209.55)
+			(xy 429.26 97.79) (xy 438.15 97.79)
 		)
 		(stroke
@@
 	(wire
 		(pts
-			(xy 454.66 279.4) (xy 473.71 279.4)
+			(xy 78.486 101.092) (xy 78.486 103.886)
 		)
 		(stroke
@@
 	(wire
 		(pts
-			(xy 608.584 105.664) (xy 613.664 105.664)
+			(xy 195.58 212.09) (xy 195.58 209.55)
 		)
 		(stroke
@@
 		)
 	)
-	(bus
+	(wire
 		(pts
-			(xy 377.19 234.95) (xy 377.19 237.49)
+			(xy 454.66 279.4) (xy 473.71 279.4)
 		)
 		(stroke
@@
 	(wire
 		(pts
-			(xy 627.38 271.78) (xy 643.89 271.78)
+			(xy 608.584 105.664) (xy 613.664 105.664)
+		)
+		(stroke
+			(width 0)
+			(type default)
+		)
+	)
+	(bus
+		(pts
+			(xy 377.19 234.95) (xy 377.19 237.49)
 		)
 		(stroke
@@
 	(wire
 		(pts
-			(xy 491.49 153.67) (xy 543.56 153.67)
+			(xy 627.38 271.78) (xy 643.89 271.78)
 		)
 		(stroke
@@
 	(wire
 		(pts
-			(xy 81.026 88.138) (xy 62.992 88.138)
+			(xy 491.49 153.67) (xy 543.56 153.67)
 		)
 		(stroke
@@
 	(wire
 		(pts
-			(xy 62.992 88.138) (xy 62.992 89.408)
-		)
-		(stroke
-			(width 0)
-			(type default)
-		)
-	)
-	(wire
-		(pts
 			(xy 735.33 252.73) (xy 721.36 252.73)
 		)
@@
 	(wire
 		(pts
-			(xy 62.992 89.408) (xy 78.486 89.408)
-		)
-		(stroke
-			(width 0)
-			(type default)
-		)
-	)
-	(wire
-		(pts
 			(xy 431.8 313.69) (xy 431.8 190.5)
 		)
@@
 	(wire
 		(pts
-			(xy 62.992 89.408) (xy 62.992 90.678)
+			(xy 95.504 102.616) (xy 95.504 110.744)
 		)
 		(stroke
@@
 	(wire
 		(pts
-			(xy 62.992 86.868) (xy 62.992 88.138)
-		)
-		(stroke
-			(width 0)
-			(type default)
-		)
-	)
-	(wire
-		(pts
 			(xy 574.04 262.89) (xy 574.04 264.16)
 		)
@@
 	(wire
 		(pts
-			(xy 81.026 88.138) (xy 81.026 103.886)
-		)
-		(stroke
-			(width 0)
-			(type default)
-		)
-	)
-	(wire
-		(pts
 			(xy 459.74 105.41) (xy 459.74 90.17)
 		)
@@
 	(wire
 		(pts
+			(xy 81.026 103.886) (xy 81.026 102.616)
+		)
+		(stroke
+			(width 0)
+			(type default)
+		)
+	)
+	(wire
+		(pts
 			(xy 693.42 254.254) (xy 694.436 255.27)
 		)
@@
 	(wire
 		(pts
+			(xy 95.504 118.364) (xy 95.504 124.206)
+		)
+		(stroke
+			(width 0)
+			(type default)
+		)
+	)
+	(wire
+		(pts
 			(xy 483.87 80.01) (xy 483.87 78.74)
 		)
@@
 	(wire
 		(pts
-			(xy 78.486 89.408) (xy 78.486 103.886)
-		)
-		(stroke
-			(width 0)
-			(type default)
-		)
-	)
-	(wire
-		(pts
 			(xy 626.364 87.884) (xy 636.524 87.884)
 		)
@@
 		(in_pos_files yes)
 		(dnp no)
-		(fields_autoplaced yes)
 		(property "Reference" "U15"
-			(at 97.536 102.5458 0)
+			(at 72.644 104.648 0)
 			(show_name no)
 			(do_not_autoplace no)
@@
 		)
 		(property "Value" "DS1302Z+"
-			(at 97.536 105.0858 0)
+			(at 87.63 123.19 0)
 			(show_name no)
 			(do_not_autoplace no)
@@
 	(symbol
 		(lib_id "power:+5V")
-		(at 62.992 86.868 0)
+		(at 78.486 101.092 0)
 		(unit 1)
 		(body_style 1)
@@
 		(fields_autoplaced yes)
 		(property "Reference" "#PWR094"
-			(at 62.992 90.678 0)
+			(at 78.486 104.902 0)
 			(hide yes)
 			(show_name no)
@@
 		)
 		(property "Value" "+5V"
-			(at 62.992 81.788 0)
+			(at 78.486 96.012 0)
 			(show_name no)
 			(do_not_autoplace no)
@@
 		)
 		(property "Footprint" ""
-			(at 62.992 86.868 0)
+			(at 78.486 101.092 0)
 			(hide yes)
 			(show_name no)
@@
 		)
 		(property "Datasheet" ""
-			(at 62.992 86.868 0)
+			(at 78.486 101.092 0)
 			(hide yes)
 			(show_name no)
@@
 		)
 		(property "Description" "Power symbol creates a global label with name \"+5V\""
-			(at 62.992 86.868 0)
+			(at 78.486 101.092 0)
 			(hide yes)
 			(show_name no)
@@
 		(in_pos_files yes)
 		(dnp no)
-		(fields_autoplaced yes)
 		(property "Reference" "U17"
-			(at 77.216 138.43 0)
+			(at 71.374 139.954 0)
 			(show_name no)
 			(do_not_autoplace no)
@@
 			)
 		)
-		(property "Value" ""
-			(at 77.216 153.67 0)
+		(property "Value" "TC1232"
+			(at 73.152 154.94 0)
 			(show_name no)
 			(do_not_autoplace no)
@@
 	(symbol
 		(lib_id "Device:C_Polarized")
-		(at 62.992 94.488 0)
+		(at 95.504 114.554 0)
 		(unit 1)
 		(body_style 1)
@@
 		(dnp no)
 		(property "Reference" "C3"
-			(at 63.754 92.202 0)
+			(at 96.266 112.268 0)
 			(show_name no)
 			(do_not_autoplace no)
@@
 			)
 		)
-		(property "Value" "0F1"
-			(at 64.008 97.282 0)
+		(property "Value" "0F1 SUPERCAP"
+			(at 96.52 117.348 0)
 			(show_name no)
 			(do_not_autoplace no)
@@
 		)
 		(property "Footprint" ""
-			(at 63.9572 98.298 0)
+			(at 96.4692 118.364 0)
 			(hide yes)
 			(show_name no)
@@
 		)
 		(property "Datasheet" ""
-			(at 62.992 94.488 0)
+			(at 95.504 114.554 0)
 			(hide yes)
 			(show_name no)
@@
 		)
 		(property "Description" "Polarized capacitor"
-			(at 62.992 94.488 0)
+			(at 95.504 114.554 0)
 			(hide yes)
 			(show_name no)
@@
 	(symbol
 		(lib_id "power:GND")
-		(at 62.992 98.298 0)
+		(at 95.504 124.206 0)
 		(unit 1)
 		(body_style 1)
@@
 		(fields_autoplaced yes)
 		(property "Reference" "#PWR036"
-			(at 62.992 104.648 0)
+			(at 95.504 130.556 0)
 			(hide yes)
 			(show_name no)
@@
 		)
 		(property "Value" "GND"
-			(at 62.992 103.378 0)
+			(at 95.504 129.286 0)
 			(show_name no)
 			(do_not_autoplace no)
@@
 		)
 		(property "Footprint" ""
-			(at 62.992 98.298 0)
+			(at 95.504 124.206 0)
 			(hide yes)
 			(show_name no)
@@
 		)
 		(property "Datasheet" ""
-			(at 62.992 98.298 0)
+			(at 95.504 124.206 0)
 			(hide yes)
 			(show_name no)
@@
 		)
 		(property "Description" "Power symbol creates a global label with name \"GND\" , ground"
-			(at 62.992 98.298 0)
+			(at 95.504 124.206 0)
 			(hide yes)
 			(show_name no)

Commit message: 4094 and 4051 implemented + update schematic to better quality and separate sheets
Parts:
- removed J10: HP, Connector_Molex:Molex_Mini-Fit_Sr_42819-22XX_1x02_P10.00mm_Vertical_ThermalVias, symbol Connector:Conn_01x02_Pin
- removed J11: GT11, Connector_Molex:Molex_Mini-Fit_Sr_42819-22XX_1x02_P10.00mm_Vertical_ThermalVias, symbol Connector:Conn_01x02_Pin
- removed J12: GT10, Connector_Molex:Molex_Mini-Fit_Sr_42819-22XX_1x02_P10.00mm_Vertical_ThermalVias, symbol Connector:Conn_01x02_Pin
- removed J13: GT8, Connector_Molex:Molex_Mini-Fit_Sr_42819-22XX_1x02_P10.00mm_Vertical_ThermalVias, symbol Connector:Conn_01x02_Pin
- removed J14: GT6, Connector_Molex:Molex_Mini-Fit_Sr_42819-22XX_1x02_P10.00mm_Vertical_ThermalVias, symbol Connector:Conn_01x02_Pin
- removed J15, J17: GT3, Connector_Molex:Molex_Mini-Fit_Sr_42819-22XX_1x02_P10.00mm_Vertical_ThermalVias, symbol Connector:Conn_01x02_Pin
- removed J16: GT9, Connector_Molex:Molex_Mini-Fit_Sr_42819-22XX_1x02_P10.00mm_Vertical_ThermalVias, symbol Connector:Conn_01x02_Pin
- removed J18: EXT, Connector_Molex:Molex_Mini-Fit_Sr_42819-22XX_1x02_P10.00mm_Vertical_ThermalVias, symbol Connector:Conn_01x02_Pin
- removed J19: SUMMA LARM, Connector_Molex:Molex_Mini-Fit_Sr_42819-22XX_1x02_P10.00mm_Vertical_ThermalVias, symbol Connector:Conn_01x02_Pin
- removed J20: GT5, Connector_Molex:Molex_Mini-Fit_Sr_42819-22XX_1x02_P10.00mm_Vertical_ThermalVias, symbol Connector:Conn_01x02_Pin
- removed J21: GT4, Connector_Molex:Molex_Mini-Fit_Sr_42819-22XX_1x02_P10.00mm_Vertical_ThermalVias, symbol Connector:Conn_01x02_Pin
- removed J22: ALARM_LED, Connector_Molex:Molex_Mini-Fit_Sr_42819-22XX_1x02_P10.00mm_Vertical_ThermalVias, symbol Connector:Conn_01x02_Pin
- removed J23: GT3X, Connector_Molex:Molex_Mini-Fit_Sr_42819-22XX_1x02_P10.00mm_Vertical_ThermalVias, symbol Connector:Conn_01x02_Pin
- removed J24: GT1, Connector_Molex:Molex_Mini-Fit_Sr_42819-22XX_1x02_P10.00mm_Vertical_ThermalVias, symbol Connector:Conn_01x02_Pin
- removed J25: GT2, Connector_Molex:Molex_Mini-Fit_Sr_42819-22XX_1x02_P10.00mm_Vertical_ThermalVias, symbol Connector:Conn_01x02_Pin
- removed J3: Conn_02x13_Odd_Even, symbol Connector_Generic:Conn_02x13_Odd_Even
- removed J4, J7: Conn_02x08_Odd_Even, symbol Connector_Generic:Conn_02x08_Odd_Even
- removed J5, J6: Conn_02x05_Odd_Even, symbol Connector_Generic:Conn_02x05_Odd_Even
- removed J8: DE9_Pins_MountingHoles, Connector_Dsub:DSUB-9_Pins_Vertical_P2.77x2.84mm_MountingHoles, symbol Connector:DE9_Pins_MountingHoles
- removed J9: LP, Connector_Molex:Molex_Mini-Fit_Sr_42819-22XX_1x02_P10.00mm_Vertical_ThermalVias, symbol Connector:Conn_01x02_Pin
- U4: value 27512 -> 27SF512
Other:
- note removed: "External Sensors/Ext Ctrl Inp/Larm Output - PCB"
- note removed: "FLEX_CABLE"
- note removed: "Internal Sensors/Service Port - PCB"
- moved on the sheet: C1, C10, C11, C12, C13, C14, C15, C16, C17, C18, C19, C2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
